File: boards/esp32/hardware/pcb/smbpcb.kicad_sch (KiCad schematic)
At the start: 64 parts, among them IC1 MiCS-6814, J1 USB_B_Micro, J2 PMS7003, Q1 SUD08P06-155L, SW1 RESET, SW2 RESET, U1 MCP73831-2-OT, U2 SGM6603-5.0YN6G_TR, U3 ESP32-WROOM-32, U4 SSD1306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

Commit message: minor
Parts:
- removed R22, R23: 10k, Capacitor_SMD:C_0805_2012Metric, symbol Device:R
Connections:
- no-connect marks 24 -> 26
Other:
- note removed: "PMS7003"
Changed lines of the file:
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@@
   (junction (at 215.138 120.65) (diameter 0.9144) (color 0 0 0 0))
   (junction (at 222.885 120.65) (diameter 0.9144) (color 0 0 0 0))
-  (junction (at 251.46 167.005) (diameter 0.9144) (color 0 0 0 0))
   (junction (at 252.476 60.96) (diameter 0.9144) (color 0 0 0 0))
   (junction (at 252.476 62.23) (diameter 0.9144) (color 0 0 0 0))
@@
   (no_connect (at 196.85 105.41))
   (no_connect (at 196.85 135.89))
+  (no_connect (at 246.38 200.025))
   (no_connect (at 248.92 200.025))
+  (no_connect (at 251.46 187.325))
   (no_connect (at 251.46 200.025))
   (no_connect (at 351.282 121.412))
@@
     (stroke (width 0) (type solid) (color 0 0 0 0))
   )
-  (wire (pts (xy 240.665 167.005) (xy 251.46 167.005))
-    (stroke (width 0) (type solid) (color 0 0 0 0))
-  )
-  (wire (pts (xy 240.665 175.26) (xy 240.665 167.005))
-    (stroke (width 0) (type solid) (color 0 0 0 0))
-  )
-  (wire (pts (xy 240.665 200.025) (xy 240.665 182.88))
-    (stroke (width 0) (type solid) (color 0 0 0 0))
-  )
   (wire (pts (xy 242.316 40.64) (xy 242.316 54.61))
     (stroke (width 0) (type solid) (color 0 0 0 0))
@@
     (stroke (width 0) (type solid) (color 0 0 0 0))
   )
-  (wire (pts (xy 246.38 200.025) (xy 240.665 200.025))
-    (stroke (width 0) (type solid) (color 0 0 0 0))
-  )
   (wire (pts (xy 247.396 40.64) (xy 247.396 44.45))
     (stroke (width 0) (type solid) (color 0 0 0 0))
@@
     (stroke (width 0) (type solid) (color 0 0 0 0))
   )
-  (wire (pts (xy 251.46 166.37) (xy 251.46 167.005))
-    (stroke (width 0) (type solid) (color 0 0 0 0))
-  )
-  (wire (pts (xy 251.46 167.005) (xy 251.46 175.26))
-    (stroke (width 0) (type solid) (color 0 0 0 0))
-  )
-  (wire (pts (xy 251.46 182.88) (xy 251.46 187.325))
-    (stroke (width 0) (type solid) (color 0 0 0 0))
-  )
   (wire (pts (xy 252.476 40.64) (xy 252.476 54.61))
     (stroke (width 0) (type solid) (color 0 0 0 0))
@@
     (effects (font (size 3 3)) (justify right bottom))
   )
-  (text "PMS7003 \n\n\n" (at 273.05 169.418 180)
-    (effects (font (size 3 3)) (justify right bottom))
-  )
   (text "OLED\n" (at 281.94 22.86 180)
     (effects (font (size 3 3)) (justify right bottom))
@@
     (pin "1")
   )
-  (symbol (lib_id "power:+3V3") (at 251.46 166.37 0) (unit 1)
-    (in_bom yes) (on_board yes)
-    (property "Reference" "#PWR0126" (id 0) (at 251.46 170.18 0)
-      (effects (font (size 1.27 1.27)) hide)
-    )
-    (property "Value" "+3V3" (id 1) (at 252.73 161.29 0))
-    (property "Footprint" "" (id 2) (at 251.46 166.37 0)
-      (effects (font (size 1.27 1.27)) hide)
-    )
-    (property "Datasheet" "" (id 3) (at 251.46 166.37 0)
-      (effects (font (size 1.27 1.27)) hide)
-    )
-    (pin "1")
-  )
   (symbol (lib_id "power:+5V") (at 265.43 117.475 90) (unit 1)
     (in_bom yes) (on_board yes)
@@
     (pin "2")
   )
-  (symbol (lib_id "Device:R") (at 240.665 179.07 0) (unit 1)
-    (in_bom yes) (on_board yes)
-    (property "Reference" "R22" (id 0) (at 236.855 175.26 0)
-      (effects (font (size 1.27 1.27)) (justify left))
-    )
-    (property "Value" "10k" (id 1) (at 235.585 177.8 0)
-      (effects (font (size 1.27 1.27)) (justify left))
-    )
-    (property "Footprint" "Capacitor_SMD:C_0805_2012Metric" (id 2) (at 238.887 179.07 90)
-      (effects (font (size 1.27 1.27)) hide)
-    )
-    (property "Datasheet" "~" (id 3) (at 240.665 179.07 0)
-      (effects (font (size 1.27 1.27)) hide)
-    )
-    (property "LCSC" "C269724" (id 4) (at 240.665 179.07 0)
-      (effects (font (size 1.27 1.27)) hide)
-    )
-    (property "Mouser" " 71-TNPU080510K0AWEN " (id 5) (at 240.665 179.07 0)
-      (effects (font (size 1.27 1.27)) hide)
-    )
-    (pin "1")
-    (pin "2")
-  )
-  (symbol (lib_id "Device:R") (at 251.46 179.07 180) (unit 1)
-    (in_bom yes) (on_board yes)
-    (property "Reference" "R23" (id 0) (at 255.27 182.88 0)
-      (effects (font (size 1.27 1.27)) (justify left))
-    )
-    (property "Value" "10k" (id 1) (at 256.54 180.34 0)
-      (effects (font (size 1.27 1.27)) (justify left))
-    )
-    (property "Footprint" "Capacitor_SMD:C_0805_2012Metric" (id 2) (at 253.238 179.07 90)
-      (effects (font (size 1.27 1.27)) hide)
-    )
-    (property "Datasheet" "~" (id 3) (at 251.46 179.07 0)
-      (effects (font (size 1.27 1.27)) hide)
-    )
-    (property "LCSC" "C269724" (id 4) (at 251.46 179.07 0)
-      (effects (font (size 1.27 1.27)) hide)
-    )
-    (property "Mouser" " 71-TNPU080510K0AWEN " (id 5) (at 251.46 179.07 0)
-      (effects (font (size 1.27 1.27)) hide)
-    )
-    (pin "1")
-    (pin "2")
-  )
   (symbol (lib_id "Device:R") (at 279.146 62.23 90) (unit 1)
     (in_bom yes) (on_board yes)
@@
       (reference "#PWR0125") (unit 1) (value "GND") (footprint "")
     )
-    (path "/f3f70168-a2da-4aae-855a-4c5a3458150a"
-      (reference "#PWR0126") (unit 1) (value "+3V3") (footprint "")
-    )
     (path "/5da8bbdd-d1a6-44ef-b955-98785bcf2cc9"
       (reference "#PWR0127") (unit 1) (value "GND") (footprint "")
@@
       (reference "R20") (unit 1) (value "130") (footprint "Capacitor_SMD:C_0805_2012Metric")
     )
-    (path "/026bd94d-e02a-47ba-bb0a-a81a59b74051"
-      (reference "R22") (unit 1) (value "10k") (footprint "Capacitor_SMD:C_0805_2012Metric")
-    )
-    (path "/860bb2e1-7ddb-481a-9248-8da6b7b007b5"
-      (reference "R23") (unit 1) (value "10k") (footprint "Capacitor_SMD:C_0805_2012Metric")
-    )
     (path "/967168fb-e7d3-45f6-8cc6-1e9e96844b85"
